File: Display/ARDUINO .brd (EAGLE design)
At the start: 181.3 x 79.6 mm, 5 parts, among them U1 ARDUINO-UNO-R3-SHIELD, U2 LCD-16X2JHD-162A

Commit message: alteração
Parts:
- moved RPOT1 2.53 mm to (173.6, 72.7)
Other:
- board size 181.3 x 79.6 mm -> 181.3 x 79.7 mm
Changed lines of the file:
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@@
 <plain>
 <wire x1="0" y1="0" x2="181.32256441284864" y2="0" width="0" layer="20"/>
-<wire x1="181.32256441284864" y1="0" x2="181.32256441284864" y2="79.58592864870052" width="0" layer="20"/>
-<wire x1="181.32256441284864" y1="79.58592864870052" x2="0" y2="79.58592864870052" width="0" layer="20"/>
-<wire x1="0" y1="79.58592864870052" x2="0" y2="0" width="0" layer="20"/>
+<wire x1="181.32256441284864" y1="0" x2="181.32256441284864" y2="79.71627133356152" width="0" layer="20"/>
+<wire x1="181.32256441284864" y1="79.71627133356152" x2="0" y2="79.71627133356152" width="0" layer="20"/>
+<wire x1="0" y1="79.71627133356152" x2="0" y2="0" width="0" layer="20"/>
 </plain>
 <attributes/>
@@
 <element name="U1" library="Tinkercad" package="ARDUINO-UNO-R3-SHIELD" package3d_urn="urn:adsk.eagle:package:32092383/3" value="ARDUINO-UNO-R3-SHIELD" x="47.885" y="29.845" rot="R270" smashed="yes"/>
 <element name="U2" library="Tinkercad" package="JHD-162A" package3d_urn="urn:adsk.eagle:package:32395061/1" value="LCD-16X2JHD-162A" x="125.6966" y="40.2169" smashed="yes"/>
-<element name="RPOT1" library="Tinkercad" package="HA-06-SM065" package3d_urn="urn:adsk.eagle:package:31496083/1" value="250k" x="173.2035" y="70.1634" smashed="yes"/>
+<element name="RPOT1" library="Tinkercad" package="HA-06-SM065" package3d_urn="urn:adsk.eagle:package:31496083/1" value="250k" x="173.5613" y="72.6678" smashed="yes"/>
 <element name="R1" library="Tinkercad" package="RESAD1016W63L850D250B" package3d_urn="urn:adsk.eagle:package:31513020/1" value="250" x="142.2066" y="45.1699" rot="R90" smashed="yes"/>
 </elements>
@@
 <wire x1="144.7466" y1="40.2169" x2="116.8066" y2="40.2169" width="0" layer="19" extent="1-1"/>
 <wire x1="144.7466" y1="40.2169" x2="157.2187" y2="73.3121" width="0" layer="19" extent="1-1"/>
-<wire x1="170.6635" y1="67.6234" x2="157.2187" y2="73.3121" width="0" layer="19" extent="1-1"/>
+<wire x1="171.0213" y1="70.1278" x2="157.2187" y2="73.3121" width="0" layer="19" extent="1-1"/>
 </signal>
 <signal name="U1_D6">
@@
 <contactref element="R1" pad="2"/>
 <wire x1="109.1866" y1="40.2169" x2="142.2066" y2="50.2499" width="0" layer="19" extent="1-1"/>
-<wire x1="175.7435" y1="67.6234" x2="142.2066" y2="50.2499" width="0" layer="19" extent="1-1"/>
+<wire x1="176.1013" y1="70.1278" x2="142.2066" y2="50.2499" width="0" layer="19" extent="1-1"/>
 <wire x1="109.1866" y1="40.2169" x2="47.885" y2="5.715" width="0" layer="19" extent="1-1"/>
 </signal>
@@
 <contactref element="U2" pad="3"/>
 <contactref element="RPOT1" pad="2"/>
-<wire x1="111.7266" y1="40.2169" x2="173.2035" y2="72.7034" width="0" layer="19" extent="1-1"/>
+<wire x1="111.7266" y1="40.2169" x2="173.5613" y2="75.2078" width="0" layer="19" extent="1-1"/>
 </signal>
 </signals>
